File: 4x5.kicad_pcb (KiCad board)
At the start: 2 copper layers, 15 parts, among them SW1 SW_Push, U1 ATmega32U4-AU, Y1 16MHz

Commit message: finished pcb
Parts:
- added D1: D_Small, Diode_SMD:D_SOD-123, F.Cu at (179.4, 111.2)
- added D2: D_Small, Diode_SMD:D_SOD-123, F.Cu at (198.4, 111.2)
- added D3: D_Small, Diode_SMD:D_SOD-123, F.Cu at (217.5, 111.1)
- added D4: D_Small, Diode_SMD:D_SOD-123, F.Cu at (179.4, 130.2)
- added D5: D_Small, Diode_SMD:D_SOD-123, F.Cu at (198.4, 130.2)
- added D6: D_Small, Diode_SMD:D_SOD-123, F.Cu at (217.5, 130.2)
- added F1: 500mA, Fuse:Fuse_1206_3216Metric, F.Cu at (210.7, 95.0)
- added MX2: MX-NoLED, MX_Alps_Hybrid:MX-1U-NoLED, B.Cu at (206.4, 111.9)
- added MX3: MX-NoLED, MX_Alps_Hybrid:MX-1U-NoLED, B.Cu at (225.4, 111.9)
- added MX4: MX-NoLED, MX_Alps_Hybrid:MX-1U-NoLED, B.Cu at (187.3, 131.0)
- added MX5: MX-NoLED, MX_Alps_Hybrid:MX-1U-NoLED, B.Cu at (206.4, 131.0)
- added MX6: MX-NoLED, MX_Alps_Hybrid:MX-1U-NoLED, B.Cu at (225.4, 131.0)
- added R5: 5.1k, Resistor_SMD:R_0805_2012Metric, F.Cu at (204.0, 91.3)
- added R6: 5.1k, Resistor_SMD:R_0805_2012Metric, F.Cu at (208.0, 91.3)
- added USB1: HRO-TYPE-C-31-M-12, Type-C:HRO-TYPE-C-31-M-12, F.Cu at (206.3, 79.3)
- MX1: moved to B.Cu
- moved Y1 71.1 mm to (230.1, 88.4), turned to 270 degrees
- moved C2 66.8 mm to (230.1, 85.1)
- moved C3 64.3 mm to (233.0, 88.7), turned to 90 degrees
- moved C1 61.1 mm to (229.3, 100.9), turned to 225 degrees
- moved C4 59.0 mm to (232.3, 93.1), turned to 315 degrees
- moved R4 55.1 mm to (232.7, 98.4), turned to 225 degrees
- moved C6 51.5 mm to (219.2, 85.7), turned to 45 degrees
- moved C5 49.6 mm to (214.2, 99.2), turned to 315 degrees
- moved C7 45.3 mm to (217.9, 102.2), turned to 135 degrees
- moved R2 37.9 mm to (206.7, 97.0), turned to 90 degrees
- moved SW1 37.7 mm to (199.2, 98.4), turned to 180 degrees
- moved R1 35.7 mm to (213.4, 91.2), turned to 315 degrees
- moved R3 31.4 mm to (204.8, 97.0), turned to 90 degrees
- moved U1 27.7 mm to (223.0, 95.2), turned to 135 degrees
- moved MX1 3.18 mm to (187.3, 111.9), turned to 180 degrees
Connections:
- MX1 pad 1: Net-(MX1-Pad1) -> col0
- U1 pad 26: Net-(U1-Pad26) -> row1
- U1 pad 27: Net-(U1-Pad27) -> row0
- U1 pad 28: Net-(U1-Pad28) -> col2
- U1 pad 29: Net-(U1-Pad29) -> col1
- U1 pad 30: Net-(U1-Pad30) -> col0
Routing:
- net GND: track 0.00 -> 137.8 mm, vias 0 -> 12
- net row1: track 0.00 -> 111.5 mm, vias 0 -> 2
- net row0: track 0.00 -> 92.6 mm, vias 0 -> 2
- net +5V: track 0.00 -> 85.9 mm, vias 0 -> 2
- net col0: track 0.00 -> 62.3 mm, vias 0 -> 1
- net Net-(R4-Pad1): track 0.00 -> 45.6 mm
- net col1: track 0.00 -> 45.5 mm, vias 0 -> 1
- net col2: track 0.00 -> 44.3 mm, vias 0 -> 1
- net Net-(R3-Pad1): track 0.00 -> 29.3 mm
- net Net-(R2-Pad1): track 0.00 -> 26.1 mm
- net VCC: track 0.00 -> 14.7 mm
- net D+: track 0.00 -> 12.4 mm
- net D-: track 0.00 -> 11.1 mm
- net Net-(C2-Pad1): track 0.00 -> 7.33 mm
- net Net-(C3-Pad1): track 0.00 -> 6.90 mm
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- added copper zone on B.Cu, net GND
- added copper zone on F.Cu, net GND
Other:
- board outline added: 57.1 x 60.3 mm
- net class Default: trace_width 0.25 -> 0.254
- net class power added: clearance 0.2, trace_width 0.381, via_dia 0.8, via_drill 0.4
