File: 4x5.kicad_pcb (KiCad board)
At the start: 2 copper layers, 57.1 x 60.3 mm, 30 parts, among them SW1 SW_Push, U1 ATmega32U4-AU, Y1 16MHz

Commit message: final update
Parts:
- C2, C3: value 10uF -> 22p
Changed lines of the file:
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@@
-(kicad_pcb (version 20171130) (host pcbnew "(5.1.6)-1")
+(kicad_pcb (version 20171130) (host pcbnew "(5.1.4)-1")
   (general
     (thickness 1.6)
@@
     (pad_to_mask_clearance 0.05)
     (aux_axis_origin 0 0)
-    (visible_elements FFFFFF7F)
+    (visible_elements 7FFFFFFF)
     (pcbplotparams
       (layerselection 0x010fc_ffffffff)
@@
       (effects (font (size 1 1) (thickness 0.15)))
     )
-    (fp_text value 10uF (at 2.3645 0.6985) (layer F.Fab)
+    (fp_text value 22p (at 2.3645 0.6985) (layer F.Fab)
       (effects (font (size 1 1) (thickness 0.15)))
     )
@@
       (effects (font (size 1 1) (thickness 0.15)))
     )
-    (fp_text value 10uF (at -3.1346 -0.9779) (layer F.Fab)
-      (effects (font (size 1 1) (thickness 0.15)))
-    )
+    (fp_text value 22p (at -3.1346 -0.9779) (layer F.Fab)
+      (effects (font (size 1 1) (thickness 0.15)))
+    )
