File: 4x5.sch (KiCad schematic (older format))
At the start: 14 parts

Commit message: finished schem
Parts:
- added D1, D2, D3, D4, D5, D6: D_Small, Diode_SMD:D_SOD-123, symbol Device:D_Small
- added MX1, MX2, MX3, MX4, MX5, MX6: MX-NoLED, MX_Alps_Hybrid:MX-1U-NoLED, symbol MX_Alps_Hybrid:MX-NoLED
- C1: footprint (none) -> Capacitor_SMD:C_0805_2012Metric
- C2, C3, C4, C5, C6, C7: renamed from C?; footprint (none) -> Capacitor_SMD:C_0805_2012Metric
- R1, R2, R3: footprint (none) -> Resistor_SMD:R_0805_2012Metric
- R4: renamed from R?; footprint (none) -> Resistor_SMD:R_0805_2012Metric
- SW1: renamed from SW?; footprint (none) -> random-keyboard-parts:SKQG-1155865
- Y1: renamed from Y?; footprint (none) -> Crystal:Crystal_SMD_3225-4Pin_3.2x2.5mm
- gave numbers to parts that had none: 1
Connections:
- new net: D1.2 (A), MX1.2 (ROW)
- new net: D2.2 (A), MX2.2 (ROW)
- new net: D3.2 (A), MX3.2 (ROW)
- new net: D4.2 (A), MX4.2 (ROW)
- new net: D5.2 (A), MX5.2 (ROW)
- new net: D6.2 (A), MX6.2 (ROW)
- new net col0: MX1.1 (COL), MX4.1 (COL)
- new net col1: MX2.1 (COL), MX5.1 (COL)
- new net col2: MX3.1 (COL), MX6.1 (COL)
- new net row0: D1.1 (K), D2.1 (K), D3.1 (K)
- new net row1: D4.1 (K), D5.1 (K), D6.1 (K)

Commit message: finished pcb
Parts:
- added F1: 500mA, Fuse:Fuse_1206_3216Metric, symbol Device:Polyfuse_Small
- added R5, R6: 5.1k, Resistor_SMD:R_0805_2012Metric, symbol Device:R_Small
- added USB1: HRO-TYPE-C-31-M-12, Type-C:HRO-TYPE-C-31-M-12, symbol Type-C:HRO-TYPE-C-31-M-12
Connections:
- net +5V: now also F1.2
- net D+: now also USB1.6 (DP1), USB1.8 (DP2)
- net D-: now also USB1.5 (DN2), USB1.7 (DN1)
- net GND: now also R5.1, R6.1, USB1.1 (GND), USB1.12 (GND), USB1.13 (SHIELD)
- net col0: now also U1.30 (PB6)
- net col1: now also U1.29 (PB5)
- net col2: now also U1.28 (PB4)
- net row0: now also U1.27 (PD7)
- net row1: now also U1.26 (PD6)
- new net: R5.2, USB1.10 (CC2)
- new net: R6.2, USB1.4 (CC1)
- new net VCC: F1.1, USB1.11 (VBUS), USB1.2 (VBUS)
- no-connect marks 0 -> 2
Other:
- moved on the sheet: C4, C5, C6, C7, D1, D2, D3, D4, D5, D6, MX1, MX2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

Commit message: final update
Parts:
- C2, C3: value 10uF -> 22p
- U1: symbol MCU_Microchip_ATmega:ATmega32U4-AU -> 4x5-rescue:ATmega32U4-AU-MCU_Microchip_ATmega
Changed lines of the file:
@@
 EESchema Schematic File Version 4
+LIBS:4x5-cache
 EELAYER 30 0
 EELAYER END
@@
 Connection ~ 5700 4350
 $Comp
-L MCU_Microchip_ATmega:ATmega32U4-AU U1
+L 4x5-rescue:ATmega32U4-AU-MCU_Microchip_ATmega U1
 U 1 1 5F05AB6C
 P 7200 3550
@@
 P 5650 2150
 F 0 "C2" V 5450 2100 50  0000 L CNN
-F 1 "10uF" V 5550 2050 50  0000 L CNN
+F 1 "22p" V 5550 2050 50  0000 L CNN
 F 2 "Capacitor_SMD:C_0805_2012Metric" H 5650 2150 50  0001 C CNN
 F 3 "~" H 5650 2150 50  0001 C CNN
@@
 P 5650 2550
 F 0 "C3" V 5450 2500 50  0000 L CNN
-F 1 "10uF" V 5550 2450 50  0000 L CNN
+F 1 "22p" V 5550 2450 50  0000 L CNN
 F 2 "Capacitor_SMD:C_0805_2012Metric" H 5650 2550 50  0001 C CNN
 F 3 "~" H 5650 2550 50  0001 C CNN
